File: hardware-smart-gaz-detector.sch (KiCad schematic (older format))
At the start: 33 parts

Commit message: update schematic
Parts:
- added D?: LED, symbol Device:LED
- added R?: 10k, symbol Device:R_Small
- added R?: 562k, symbol Device:R_Small
- added SW?: SW_Push, symbol Switch:SW_Push
Connections:
- net labels added: ADC1_Temperature, PTC_Y2, RESET, RN2483_RESET
- net labels removed: ICSP_RESET, UART0_RESET, UART_RX, UART_TX, U_temperature, XCK0, nRESET
- wire segments 58 -> 61
- no-connect marks 37 -> 35
Other:
- moved on the sheet: BZ?, D?, L?, Q?, R?, U?

Commit message: version 0.2
Parts:
- removed C?: 4.7µF, symbol Device:C_Small
- removed U?: TPL5111, Package_TO_SOT_SMD:SOT-23-6, symbol Timer:TPL5111
- removed U?: MCP1640CH, Package_TO_SOT_SMD:SOT-23-6, symbol Regulator_Switching:MCP1640CH
- removed U?: ATmega328PB-AU, Package_QFP:TQFP-32_7x7mm_P0.8mm, symbol MCU_Microchip_ATmega:ATmega328PB-AU
- added C11: 1µ, symbol Device:C_Small
- added C12, C8: 100n, symbol Device:C_Small
- added C2: 100nF, symbol Device:C_Small
- added Q1, Q4: SI2301CDS-T1-GE3, Vishay-S-03946-07_2001-K-*, symbol project_symbols:SI2301CDS-T1-GE3
- added Q2, Q5: Q_NPN_BCE, symbol Device:Q_NPN_BCE
- added R15, R2: 1k2, symbol Device:R_Small
- added R16, R4: 22k, symbol Device:R_Small
- added R17, R7: 100k, symbol Device:R_Small
- added U1: MCP1640BCH, Package_TO_SOT_SMD:SOT-23-6, symbol Regulator_Switching:MCP1640BCH
- added U2: TPL5010, Package_TO_SOT_SMD:SOT-23-6, symbol Timer:TPL5010
- added U4: ATmega328P-AU, Package_QFP:TQFP-32_7x7mm_P0.8mm, symbol MCU_Microchip_ATmega:ATmega328P-AU
- BT1: renamed from BT?; value Battery_Cell -> AA Battery
- L2: renamed from L?; value L_Small -> ?
- R1: renamed from R?; value 10k -> 22k
- R10: renamed from R?; value ? -> ?/1k
- R14: renamed from R?; value 562k -> 260
- gave numbers to parts that had none: 28
Connections:
- net labels added: ADC4_Battery, EN_RN2483, GPIO_AOP, GPIO_Battery, GPIO_DONE, GPIO_Gaz, GPIO_LED, GPIO_PolySi, GPIO_Temperature, RESET_RN2483, Vdd_RN2483, WAKE, nRST, u_gaz
- net labels removed: PTC_Y2, RESET, RN2483_RESET, U_gaz
- wire segments 61 -> 85
- no-connect marks 35 -> 24
Other:
- note added: "Battery measure trigger"
- note added: "LoRa Transceiver"
- note added: "Power on trigger"
- note removed: "LoRa Transmitter"
- moved on the sheet: BT1, BZ1, C1, C10, C3, C4, C5, C6, C7, C9, D1, D2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
