File: hardware-smart-gaz-detector-extension-board.sch (KiCad schematic (older format))
At the start: 63 parts, among them J1 Conn_ICSP, J2 Conn_Extension, J3 Conn_Piezo, J4 SMA, J5 USB_B_Mini, SW1 SW_Push, U1 RE46C318S8F, U2 ATmega328P-AU, U3 SGP40-D-R4, U4 SHT4x, U5 TPL5010, U6 TPS61090, U7 MCP73871-2AA

Commit message: final commit before portfolio
Parts:
- removed BT1: 1c LiPo, Connector_JST:JST_PH_B2B-PH-K_1x02_P2.00mm_Vertical, symbol Device:Battery_Cell
- removed C10, C12: 1µ, Capacitor_SMD:C_0603_1608Metric, symbol Device:C_Small
- removed C11, C13, C14, C17, C18, C7, C8: 100n, Capacitor_SMD:C_0603_1608Metric, symbol Device:C_Small
- removed C15, C16, C21, C22: 10µ, Capacitor_SMD:C_0603_1608Metric, symbol Device:C_Small
- removed C19: 2.2µ, Capacitor_SMD:C_0603_1608Metric, symbol Device:C_Small
- removed C20: 100µ, Capacitor_SMD:CP_Elec_6.3x5.8, symbol Device:CP_Small
- removed C3, C9: 4.7µ, Capacitor_SMD:C_0603_1608Metric, symbol Device:C_Small
- removed D1: D_Schottky, Diode_SMD:D_SMA, symbol Device:D_Schottky
- removed D2: LED, LED_SMD:LED_1206_3216Metric, symbol Device:LED
- removed D3: ORANGE, LED_SMD:LED_1206_3216Metric, symbol Device:LED_Small
- removed D4: GREEN, LED_SMD:LED_1206_3216Metric, symbol Device:LED_Small
- removed J1: Conn_ICSP, Connector_PinHeader_2.54mm:PinHeader_2x03_P2.54mm_Vertical, symbol Connector_Generic:Conn_02x03_Top_Bottom
- removed J2: Conn_Extension, Connector_PinSocket_2.54mm:PinSocket_2x04_P2.54mm_Vertical, symbol Connector_Generic:Conn_02x04_Top_Bottom
- removed J3: Conn_Piezo, Connector_PinSocket_2.54mm:PinSocket_1x03_P2.54mm_Vertical, symbol Connector:Conn_01x03_Male
- removed J4: SMA, Connector_Coaxial:SMA_Amphenol_132289_EdgeMount, symbol Connector:Conn_Coaxial
- removed J5: USB_B_Mini, Connector_USB:USB_Micro-B_Amphenol_10103594-0001LF_Horizontal, symbol Connector:USB_B_Mini
- removed L1: 10µ, Inductor_SMD:L_Taiyo-Yuden_MD-4040, symbol Device:L
- removed L2: 10µ, Inductor_SMD:L_0805_2012Metric, symbol Device:L
- removed L3: 6.8µ, Inductor_SMD:L_Taiyo-Yuden_MD-5050, symbol Device:L
- removed MD1: RN2483A-I_RM103, project_footprint:Microchip-RN2483A-I_RM103-0-0-MFG, symbol project_symbols:RN2483A-I_RM103
- removed R10: 330k, Resistor_SMD:R_0603_1608Metric, symbol Device:R_Small
- removed R11: 110k, Resistor_SMD:R_0603_1608Metric, symbol Device:R_Small
- removed R12, R18, R19: 1k, Resistor_SMD:R_0603_1608Metric, symbol Device:R_Small
- removed R13: 100k, Resistor_SMD:R_0603_1608Metric, symbol Device:R_Small
- removed R14: 15k, Resistor_SMD:R_0603_1608Metric, symbol Device:R_Small
- removed R15: 1.1M, Resistor_SMD:R_0603_1608Metric, symbol Device:R_Small
- removed R16: 200k, Resistor_SMD:R_0603_1608Metric, symbol Device:R_Small
- removed R17: 1M, Resistor_SMD:R_0603_1608Metric, symbol Device:R_Small
- removed R8: 1.87M, Resistor_SMD:R_0603_1608Metric, symbol Device:R_Small
- removed R9: 340k, Resistor_SMD:R_0603_1608Metric, symbol Device:R_Small
- removed SW1: SW_Push, Button_Switch_SMD:SW_Push_1P1T_NO_CK_KMR2, symbol Switch:SW_Push
- removed U1: RE46C318S8F, project_footprint:RE46C318S8F, symbol project_symbols:RE46C318S8F
- removed U2: ATmega328P-AU, Package_QFP:TQFP-32_7x7mm_P0.8mm, symbol MCU_Microchip_ATmega:ATmega328P-AU
- removed U3: SGP40-D-R4, project_footprint:Sensirion-SGP40-D-R4-MFG, symbol project_symbols:SGP40-D-R4
- removed U4: SHT4x, project_footprint:WDFN-4_1.5x1.5_Pitch0.8mm, symbol project_symbols:SHT4x
- removed U5: TPL5010, Package_TO_SOT_SMD:SOT-23-6, symbol Timer:TPL5010
- removed U6: TPS61090, Package_DFN_QFN:Texas_S-PVQFN-N16_EP2.7x2.7mm_ThermalVias, symbol Regulator_Switching:TPS61090
- removed U7: MCP73871-2AA, Package_DFN_QFN:QFN-20-1EP_4x4mm_P0.5mm_EP2.5x2.5mm, symbol Battery_Management:MCP73871-2AA
- added C3: 10µ, Capacitor_SMD:CP_Elec_5x5.4, symbol Device:CP_Small
- added J1: Conn_Extension, Connector_PinSocket_2.54mm:PinSocket_2x04_P2.54mm_Vertical, symbol Connector_Generic:Conn_02x04_Top_Bottom
- added J2: Jack-DC, Connector_BarrelJack:BarrelJack_Horizontal, symbol Connector:Jack-DC
- added Q1: FDN327N, project_footprint:ON_Semi-527AG-01-12_2008-O-0, symbol project_symbols:FDN327N
- added U1: aime_gaz_sensor, Package_TO_SOT_THT:TO-5-10_Window, symbol project_symbols:AIME_GAZ_SENSOR
- added U2: LTC2050HVCS5TRPBF, project_footprint:Linear_Technology-LTC2050HVCS5TRPBF-Level_B, symbol project_symbols:LTC2050HVCS5TRPBF
- added U3: MCP4017-xxxxLT, Package_TO_SOT_SMD:SOT-363_SC-70-6, symbol Potentiometer_Digital:MCP4017-xxxxLT
- C2, C4: value 10µ -> 100n
- C5: value 1n -> 100n
- C6: value 100n -> 1µ
- R1: value 1.5M -> 10k
- R2: value 4.7k -> 250
- R3: value 4.7k -> 10k
- R4: value 10 -> 100k
- R5: value 200k -> 1k
- R6: value 100k -> 50k
- R7: value 22k -> 1k
Connections:
- net labels added: +12V, ADC0_Gaz, ADC1_Temperature, PWM_PolySi, aop_-, aop_out, u_gaz
- net labels removed: +10V, +3.3VA, +BATT, ADC0, ADC1, GND2, GPIO_Done, GPIO_Horn, GPIO_LBO, PCINT0_Wake, PWM0A_Led, PWM0B, RN2483_nRST, SPI_MISO, SPI_MOSI, SPI_SCK, UART0_RX, UART0_TX, VBUS, nRST, piezo_feedback, piezo_gnd, piezo_input
- wire segments 120 -> 40
- no-connect marks 42 -> 2
Other:
- note added: "Extension board"
- note removed: "Buzzer"
- note removed: "LoRa Transceiver"
- note removed: "MCU"
- note removed: "Power Management"
- note removed: "Sensors"
